File: V2/V2.kicad_pcb (KiCad board)
At the start: 2 copper layers, 183 parts, among them U1 Elite-C

Commit message: Updated schematic and pcb design
Parts:
- moved D88 622.3 mm to (675.9, 184.3)
- moved D1 622.3 mm to (702.0, 224.7)
- moved D10 622.3 mm to (782.7, 223.4)
- moved D11 622.3 mm to (765.4, 223.4)
- moved D12 622.3 mm to (771.0, 230.1)
- moved D13 622.3 mm to (925.5, 88.0)
- moved D14 622.3 mm to (776.9, 226.8)
- moved D15 622.3 mm to (776.9, 223.4)
- moved D16 622.3 mm to (924.4, 74.6)
- moved D17 622.3 mm to (765.3, 230.1)
- moved D18 622.3 mm to (771.2, 226.8)
- moved D19 622.3 mm to (771.2, 223.4)
- moved D2 622.3 mm to (788.3, 230.1)
- moved D20 622.3 mm to (924.4, 71.2)
- moved D21 622.3 mm to (924.4, 67.9)
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
Commit message: Added Edge Cuts
Parts:
- D1, D10, D11, D12, D13, D14, D15, D16, D17, D18, D19, D2, D20, D21, D22, D23, D24, D25, D26, D27, D28, D29, D3, D30, D31, D32, D33, D34, D35, D36, D37, D38, D39, D4, D40, D41, D42, D43, D44, D45, D46, D47, D48, D49, D5, D50, D51, D52, D53, D54, D55, D56, D57, D58, D59, D6, D60, D61, D62, D63, D64, D65, D66, D67, D68, D69, D7, D70, D71, D72, D73, D74, D75, D76, D77, D78, D79, D8, D80, D81, D82, D83, D84, D85, D86, D87, D88, D89, D9, D90, D91: moved to B.Cu
- moved D8 897.7 mm to (28.6, 47.6), turned to 180 degrees
- moved D9 897.0 mm to (28.6, 66.7), turned to 180 degrees
- moved D13 878.8 mm to (47.6, 47.6), turned to 180 degrees
- moved D16 860.1 mm to (66.7, 9.53), turned to 90 degrees
- moved D2 804.4 mm to (9.53, 28.6), turned to 180 degrees
- moved D4 800.1 mm to (9.53, 66.7), turned to 180 degrees
- moved D3 799.2 mm to (9.53, 47.6), turned to 180 degrees
- moved D6 785.5 mm to (28.6, 9.53), turned to 180 degrees
- moved D7 779.7 mm to (28.6, 28.6), turned to 180 degrees
- moved D12 750.9 mm to (47.6, 28.6), turned to 180 degrees
- moved D11 749.0 mm to (47.6, 9.53), turned to 180 degrees
- moved D14 746.6 mm to (47.6, 66.7), turned to 180 degrees
- moved D17 727.1 mm to (66.7, 28.5), turned to 90 degrees
- moved D1 725.1 mm to (9.53, 9.53), turned to 180 degrees
- moved D18 722.5 mm to (66.7, 66.6), turned to 90 degrees
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Other:
- board outline added: 442.2 x 112.7 mm

Commit message: Finished PCB
Parts:
- added MX92: KC_P0, MX_Alps_Hybrid:MXOnly-2U-Hotswap-ReversedStabilizers, F.Cu at (9.53, 76.2)
- moved D5 707.2 mm to (9.53, 83.2), turned to 90 degrees
- moved D10 693.9 mm to (28.6, 83.2), turned to 90 degrees
- moved D15 680.6 mm to (47.6, 83.2), turned to 90 degrees
- moved D24 643.9 mm to (119.1, 83.2), turned to 90 degrees
- moved D25 642.3 mm to (109.5, 9.53)
- moved D19 638.7 mm to (95.2, 83.2), turned to 90 degrees
- moved D22 637.2 mm to (104.8, 44.1), turned to 90 degrees
- moved D82 629.0 mm to (394.5, 9.53), turned to 90 degrees
- moved D34 628.4 mm to (151.6, 87.2), turned to 80 degrees
- moved D84 625.2 mm to (394.5, 47.3), turned to 90 degrees
- moved D28 623.4 mm to (123.8, 47.6)
- moved D31 622.2 mm to (139.2, 29.0), turned to 170 degrees
- moved D32 622.2 mm to (142.9, 49.0), turned to 170 degrees
- moved D83 621.0 mm to (394.5, 28.6), turned to 90 degrees
- moved D29 619.0 mm to (133.3, 66.7)
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Connections:
- U1 pad 1: Net-(U1-Pad1) -> Col0
- U1 pad 10: Net-(U1-Pad10) -> Col7
- U1 pad 11: Net-(U1-Pad11) -> Col8
- U1 pad 12: Net-(U1-Pad12) -> Col9
- U1 pad 13: Net-(U1-Pad13) -> Col10
- U1 pad 14: Net-(U1-Pad14) -> Col11
- U1 pad 15: Net-(U1-Pad15) -> Col12
- U1 pad 16: Net-(U1-Pad16) -> Col13
- U1 pad 17: Net-(U1-Pad17) -> Col14
- U1 pad 18: Net-(U1-Pad18) -> Col15
- U1 pad 19: Net-(U1-Pad19) -> Col16
- U1 pad 2: Net-(U1-Pad2) -> Col1
- U1 pad 20: Net-(U1-Pad20) -> Col17
- U1 pad 24: Net-(U1-Pad24) -> Col18
- U1 pad 25: Net-(U1-Pad25) -> Row0
- U1 pad 26: Net-(U1-Pad26) -> Row1
- U1 pad 28: Net-(U1-Pad28) -> Row2
- U1 pad 29: Net-(U1-Pad29) -> Row3
- U1 pad 5: Net-(U1-Pad5) -> Col2
- U1 pad 6: Net-(U1-Pad6) -> Col3
- U1 pad 7: Net-(U1-Pad7) -> Col4
- U1 pad 8: Net-(U1-Pad8) -> Col5
- U1 pad 9: Net-(U1-Pad9) -> Col6
Routing:
- net Row2: track 0.00 -> 513.5 mm, vias 0 -> 18
- net Row3: track 0.00 -> 510.4 mm, vias 0 -> 19
- net Row1: track 0.00 -> 477.3 mm, vias 0 -> 18
- net Row4: track 0.00 -> 444.9 mm, vias 0 -> 2
- net Row0: track 0.00 -> 435.2 mm, vias 0 -> 18
- net Col0: track 0.00 -> 309.5 mm
- net Col18: track 0.00 -> 306.4 mm
- net Col1: track 0.00 -> 279.3 mm
- net Col3: track 0.00 -> 272.4 mm
- net Col2: track 0.00 -> 261.2 mm
- net Col17: track 0.00 -> 255.3 mm
- net Col16: track 0.00 -> 242.9 mm
- net Col4: track 0.00 -> 231.3 mm
- net Col15: track 0.00 -> 224.4 mm, vias 0 -> 1
- net Col14: track 0.00 -> 205.0 mm, vias 0 -> 1
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