File: V2/V2.kicad_pcb (KiCad board)
At the start: 2 copper layers, 442.2 x 112.7 mm, 184 parts, among them U1 Elite-C

Commit message: Switched to LED
Parts:
- MX92: footprint MX_Alps_Hybrid:MXOnly-2U-Hotswap-ReversedStabilizers -> MX_Alps_Hybrid:MXOnly-2U-Hotswap
- moved D5 15.7 mm to (25.2, 83.2)
- turned D41 to 170 degrees
- turned D46 to 170 degrees
- turned MX92 to 180 degrees
Connections:
- U1 pad 27: Net-(U1-Pad27) -> Row4
Routing:
- net Row4: track 444.9 -> 499.5 mm, vias 2 -> 1
- net Col0: track 309.5 -> 324.5 mm, vias 0 -> 6
- net Col7: track 123.5 -> 136.6 mm, vias 1 -> 4
- net Row0: track 435.2 -> 423.9 mm, vias 18 -> 0
- net Col18: track 306.4 -> 295.8 mm, vias 0 -> 5
- net Col5: track 193.6 -> 201.3 mm, vias 1 -> 4
- net Row3: track 510.4 -> 517.6 mm, vias 19 -> 3
- net Col12: track 144.3 -> 150.8 mm, vias 1 -> 5
- net Net-(D87-Pad2): track 28.7 -> 22.3 mm
- net Col13: track 181.6 -> 187.8 mm, vias 1 -> 5
- net Col9: track 117.8 -> 123.7 mm, vias 0 -> 5
- net Col14: track 205.0 -> 210.3 mm, vias 1 -> 4
- net Col8: track 137.9 -> 133.2 mm, vias 1 -> 5
- net Col11: track 112.8 -> 108.4 mm, vias 1 -> 5
- net Col6: track 170.5 -> 174.5 mm, vias 1 -> 5
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
Commit message: Update V2.kicad_pcb
Parts:
- MX1, MX10, MX11, MX12, MX13, MX14, MX15, MX16, MX2, MX20, MX25, MX26, MX27, MX28, MX29, MX3, MX30, MX31, MX32, MX33, MX35, MX36, MX37, MX38, MX39, MX4, MX40, MX41, MX42, MX44, MX45, MX46, MX47, MX48, MX49, MX5, MX50, MX51, MX52, MX53, MX54, MX55, MX56, MX58, MX59, MX6, MX60, MX61, MX63, MX64, MX65, MX66, MX68, MX69, MX7, MX70, MX72, MX73, MX74, MX75, MX77, MX78, MX79, MX8, MX81, MX85, MX86, MX87, MX88, MX89, MX9, MX90, MX91: footprint MX_Alps_Hybrid:MXOnly-1U-Hotswap -> MX_Alps_Hybrid:MXOnly-1U
- MX17, MX18, MX82: footprint MX_Alps_Hybrid:MXOnly-2U-Hotswap -> MX_Alps_Hybrid:MXOnly-2U
- MX19, MX24, MX34, MX62, MX67, MX71, MX76: footprint MX_Alps_Hybrid:MXOnly-1.25U-Hotswap -> MX_Alps_Hybrid:MXOnly-1.25U
- MX21, MX83: footprint MX_Alps_Hybrid:MXOnly-1.5U-Hotswap -> MX_Alps_Hybrid:MXOnly-1.5U
- MX22, MX80: footprint MX_Alps_Hybrid:MXOnly-1.75U-Hotswap -> MX_Alps_Hybrid:MXOnly-1.75U
- MX23, MX84: footprint MX_Alps_Hybrid:MXOnly-2.25U-Hotswap -> MX_Alps_Hybrid:MXOnly-2.25U
- MX43: footprint MX_Alps_Hybrid:MXOnly-2.25U-Hotswap-ReversedStabilizers -> MX_Alps_Hybrid:MXOnly-2.25U-ReversedStabilizers
- MX57: footprint MX_Alps_Hybrid:MXOnly-2.75U-Hotswap-ReversedStabilizers -> MX_Alps_Hybrid:MXOnly-2.75U-ReversedStabilizers
- MX92: footprint MX_Alps_Hybrid:MXOnly-2U-Hotswap -> MX_Alps_Hybrid:MXOnly-2U-ReversedStabilizers
- turned MX92 to 0 degrees
Routing:
- net Col0: track 324.5 -> 300.1 mm, vias 6 -> 0
- net Col9: track 123.7 -> 103.9 mm, vias 5 -> 0
- net Col5: track 201.3 -> 185.0 mm, vias 4 -> 0
- net Row2: track 515.6 -> 502.7 mm
- net Col18: track 295.8 -> 308.0 mm, vias 5 -> 1
- net Col3: track 271.6 -> 261.3 mm, vias 3 -> 0
- net Col7: track 136.6 -> 126.6 mm, vias 4 -> 0
- net Col16: track 240.2 -> 250.1 mm, vias 5 -> 0
- net Col6: track 174.5 -> 165.7 mm, vias 5 -> 0
- net Col11: track 108.4 -> 116.6 mm, vias 5 -> 1
- net Col4: track 231.7 -> 224.0 mm, vias 5 -> 0
- net Col1: track 278.9 -> 271.4 mm, vias 5 -> 0
- net Col15: track 223.5 -> 230.9 mm, vias 5 -> 0
- net Col17: track 253.9 -> 260.3 mm, vias 5 -> 0
- net Net-(D57-Pad2): track 39.0 -> 32.8 mm
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
Commit message: Update PCB
Parts:
- MX1, MX10, MX11, MX12, MX13, MX14, MX15, MX16, MX2, MX20, MX25, MX26, MX27, MX28, MX29, MX3, MX30, MX31, MX32, MX33, MX35, MX36, MX37, MX38, MX39, MX4, MX40, MX41, MX42, MX44, MX45, MX46, MX47, MX48, MX49, MX5, MX50, MX51, MX52, MX53, MX54, MX55, MX56, MX58, MX59, MX6, MX60, MX61, MX63, MX64, MX65, MX66, MX68, MX69, MX7, MX70, MX72, MX73, MX74, MX75, MX77, MX78, MX79, MX8, MX81, MX85, MX86, MX87, MX88, MX89, MX9, MX90, MX91: footprint MX_Alps_Hybrid:MXOnly-1U -> MX_Alps_Hybrid:MXOnly-1U-NoLED
- MX17, MX18: footprint MX_Alps_Hybrid:MXOnly-2U -> MX_Alps_Hybrid:MXOnly-2U-NoLED
- MX19, MX24, MX34, MX62, MX67, MX71, MX76: footprint MX_Alps_Hybrid:MXOnly-1.25U -> MX_Alps_Hybrid:MXOnly-1.25U-NoLED
- MX21, MX83: footprint MX_Alps_Hybrid:MXOnly-1.5U -> MX_Alps_Hybrid:MXOnly-1.5U-NoLED
- MX22, MX80: footprint MX_Alps_Hybrid:MXOnly-1.75U -> MX_Alps_Hybrid:MXOnly-1.75U-NoLED
- MX23, MX84: footprint MX_Alps_Hybrid:MXOnly-2.25U -> MX_Alps_Hybrid:MXOnly-2.25U-NoLED
- MX43: footprint MX_Alps_Hybrid:MXOnly-2.25U-ReversedStabilizers -> MX_Alps_Hybrid:MXOnly-2.25U-ReversedStabilizers-NoLED
- MX57: footprint MX_Alps_Hybrid:MXOnly-2.75U-ReversedStabilizers -> MX_Alps_Hybrid:MXOnly-2.75U-ReversedStabilizers-NoLED
- MX82: footprint MX_Alps_Hybrid:MXOnly-2U -> MX_Alps_Hybrid:MXOnly-2U-ReversedStabilizers-NoLED
- MX92: footprint MX_Alps_Hybrid:MXOnly-2U-ReversedStabilizers -> MX_Alps_Hybrid:MXOnly-2U-ReversedStabilizers-NoLED
- moved D84 42.9 mm to (351.7, 47.6)
- moved D82 38.1 mm to (356.4, 9.53)
- moved D80 33.3 mm to (342.2, 66.7), turned to 90 degrees
- moved D83 28.6 mm to (366.0, 28.6)
- moved D27 19.6 mm to (114.3, 47.6), turned to 90 degrees
- moved D17 19.1 mm to (66.7, 47.6)
- moved D69 19.1 mm to (308.8, 28.5), turned to 90 degrees
- moved D72 19.1 mm to (318.3, 9.53), turned to 90 degrees
- moved D73 19.1 mm to (327.9, 28.6), turned to 90 degrees
- moved D77 19.1 mm to (337.4, 9.53), turned to 90 degrees
- moved D85 19.1 mm to (375.5, 66.7), turned to 90 degrees
- moved D68 19.1 mm to (299.3, 9.53), turned to 90 degrees
- moved D78 19.1 mm to (346.9, 28.6), turned to 90 degrees
- moved D90 19.1 mm to (394.5, 66.7), turned to 90 degrees
- moved D28 19.0 mm to (123.8, 66.7), turned to 90 degrees
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Routing:
- net Row3: track 514.8 -> 465.2 mm
- net Row2: track 502.7 -> 458.4 mm
- net Row4: track 501.9 -> 477.8 mm
- net Net-(D28-Pad2): track 16.8 -> 34.9 mm, vias 0 -> 1
- net Net-(D27-Pad2): track 16.8 -> 33.0 mm, vias 0 -> 1
- net Col17: track 260.3 -> 275.2 mm
- net Net-(D17-Pad2): track 15.9 -> 30.4 mm, vias 0 -> 1
- net Net-(D29-Pad2): track 16.8 -> 30.4 mm
- net Col13: track 192.0 -> 179.3 mm
- net Col18: track 308.0 -> 296.9 mm, vias 1 -> 0
- net Col12: track 156.4 -> 146.7 mm
- net Col15: track 230.9 -> 222.0 mm
- net Net-(D47-Pad2): track 8.41 -> 15.9 mm
- net Col16: track 250.1 -> 257.3 mm
- net Col11: track 116.6 -> 123.1 mm, vias 1 -> 0
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- added copper zone on B.Cu, net (none)
- added copper zone on F.Cu, net (none)
