File: V2/V2.kicad_pcb (KiCad board)
At the start: 2 copper layers, 442.2 x 112.7 mm, 184 parts, among them U1 Elite-C

Commit message: Complete Redesign
Parts:
- added D92: D_Small, Diode_SMD:D_SOD-123, B.Cu at (421.4, 83.3)
- added SW1: Rotary_Encoder_Switch, Keebio-Parts:RotaryEncoder_Alps_EC11E-Switch_Vertical_H20mm, F.Cu at (430.9, 0.00)
- MX1: value KC_NLCK -> Num Lock
- MX10: value KC_P0 -> PAST
- MX11: value KC_PAST -> P8
- MX12: value KC_P9 -> P9
- MX13: value KC_P6 -> P5
- MX14: value KC_P3 -> P6
- MX15: value KC_PDOT -> P3
- MX16: value KC_PMNS -> PDOT
- MX17: value KC_PPLS -> PMINUS; footprint MX_Alps_Hybrid:MXOnly-2U-NoLED -> MX_Alps_Hybrid:MXOnly-1U-NoLED
- MX18: value KC_PENT -> PPLS
- MX19: value KC_LCTL -> PENT; footprint MX_Alps_Hybrid:MXOnly-1.25U-NoLED -> MX_Alps_Hybrid:MXOnly-2U-NoLED
- MX2: value KC_P7 -> P7
- MX20: value KC_ESC -> LCTRL; footprint MX_Alps_Hybrid:MXOnly-1U-NoLED -> MX_Alps_Hybrid:MXOnly-1.25U-NoLED
- MX21: value KC_TAB -> LSHFT; footprint MX_Alps_Hybrid:MXOnly-1.5U-NoLED -> MX_Alps_Hybrid:MXOnly-2U-NoLED
- MX22: value KC_CAPS -> CAPS
- MX23: value KC_LSFT -> Tab; footprint MX_Alps_Hybrid:MXOnly-2.25U-NoLED -> MX_Alps_Hybrid:MXOnly-1.25U-NoLED
- MX24: value KC_LGUI -> ESC; footprint MX_Alps_Hybrid:MXOnly-1.25U-NoLED -> MX_Alps_Hybrid:MXOnly-1U-NoLED
- MX25: value KC_GRV -> GRV
- MX26: value KC_1 -> Q
- MX27: value KC_Q -> A
- MX28: value KC_A -> Z
- MX29: value KC_Z -> LGUI; footprint MX_Alps_Hybrid:MXOnly-1U-NoLED -> MX_Alps_Hybrid:MXOnly-1.25U-NoLED
- MX3: value KC_P4 -> P4
- MX30: value KC_2 -> LALT; footprint MX_Alps_Hybrid:MXOnly-1U-NoLED -> MX_Alps_Hybrid:MXOnly-1.25U-NoLED
- MX31: value KC_W -> X
- MX32: value KC_S -> S
- MX33: value KC_X -> 1
- MX34: value KC_LALT -> 2; footprint MX_Alps_Hybrid:MXOnly-1.25U-NoLED -> MX_Alps_Hybrid:MXOnly-1U-NoLED
- MX35: value KC_3 -> W
- MX36: value KC_E -> E
- MX37: value KC_D -> D
- MX38: value KC_C -> C
- MX39: value KC_4 -> Space; footprint MX_Alps_Hybrid:MXOnly-1U-NoLED -> MX_Alps_Hybrid:MXOnly-2.25U-ReversedStabilizers-NoLED
- MX4: value KC_P1 -> P1
- MX40: value KC_R -> V
- MX41: value KC_F -> 3
- MX42: value KC_V -> 4
- MX43: value KC_SPC -> R; footprint MX_Alps_Hybrid:MXOnly-2.25U-ReversedStabilizers-NoLED -> MX_Alps_Hybrid:MXOnly-1U-NoLED
- MX44: value KC_5 -> F
- MX45: value KC_T -> B
- MX46: value KC_G -> G
- MX47: value KC_B -> T
- MX48: value LT(1, KC_SPC) -> 5
- MX49: value KC_6 -> 6
- MX5: value KC_P0 -> P0; footprint MX_Alps_Hybrid:MXOnly-1U-NoLED -> MX_Alps_Hybrid:MXOnly-2U-ReversedStabilizers-NoLED
- MX50: value KC_Y -> Y
- MX51: value KC_H -> H
- MX52: value KC_B -> B-2
- MX53: value KC_7 -> Fn
- MX54: value KC_U -> Space Right; footprint MX_Alps_Hybrid:MXOnly-1U-NoLED -> MX_Alps_Hybrid:MXOnly-2.75U-ReversedStabilizers-NoLED
- MX55: value KC_J -> N
- MX56: value KC_N -> J
- MX57: value KC_SPC -> 7; footprint MX_Alps_Hybrid:MXOnly-2.75U-ReversedStabilizers-NoLED -> MX_Alps_Hybrid:MXOnly-1U-NoLED
- MX58: value KC_8 -> 8
- MX59: value KC_I -> U
- MX6: value KC_PSLS -> P0
- MX60: value KC_K -> I
- MX61: value KC_M -> K
- MX62: value KC_RALT -> M; footprint MX_Alps_Hybrid:MXOnly-1.25U-NoLED -> MX_Alps_Hybrid:MXOnly-1U-NoLED
- MX63: value KC_9 -> RALT; footprint MX_Alps_Hybrid:MXOnly-1U-NoLED -> MX_Alps_Hybrid:MXOnly-1.25U-NoLED
- MX64: value KC_O -> <
- MX65: value KC_L -> 9
- MX66: value KC_COMM -> O
- MX67: value KC_RGUI -> L; footprint MX_Alps_Hybrid:MXOnly-1.25U-NoLED -> MX_Alps_Hybrid:MXOnly-1U-NoLED
- MX68: value KC_0 -> >
- MX69: value KC_P -> RGUI; footprint MX_Alps_Hybrid:MXOnly-1U-NoLED -> MX_Alps_Hybrid:MXOnly-1.25U-NoLED
- MX7: value KC_P8 -> P0
- MX70: value KC_DOT -> APP; footprint MX_Alps_Hybrid:MXOnly-1U-NoLED -> MX_Alps_Hybrid:MXOnly-1.25U-NoLED
- MX71: value KC_APP -> ?; footprint MX_Alps_Hybrid:MXOnly-1.25U-NoLED -> MX_Alps_Hybrid:MXOnly-1U-NoLED
- MX72: value KC_MINS -> :
- MX73: value KC_LBRC -> 0
- MX74: value KC_SCLN -> -
- MX75: value KC_SLSH -> P
- MX76: value KC_RCTL -> [; footprint MX_Alps_Hybrid:MXOnly-1.25U-NoLED -> MX_Alps_Hybrid:MXOnly-1U-NoLED
- MX77: value KC_EQL -> '
- MX78: value KC_RBRC -> RSHFT; footprint MX_Alps_Hybrid:MXOnly-1U-NoLED -> MX_Alps_Hybrid:MXOnly-2.25U-NoLED
- MX79: value KC_QUOT -> RCTRL; footprint MX_Alps_Hybrid:MXOnly-1U-NoLED -> MX_Alps_Hybrid:MXOnly-1.25U-NoLED
- MX8: value KC_P5 -> P2
- MX80: value KC_RSFT -> Left; footprint MX_Alps_Hybrid:MXOnly-1.75U-NoLED -> MX_Alps_Hybrid:MXOnly-1U-NoLED
- MX81: value KC_LEFT -> =
- MX82: value KC_BSPC -> Backspace; footprint MX_Alps_Hybrid:MXOnly-2U-ReversedStabilizers-NoLED -> MX_Alps_Hybrid:MXOnly-2U-NoLED
- MX83: value KC_BSLS -> ]; footprint MX_Alps_Hybrid:MXOnly-1.5U-NoLED -> MX_Alps_Hybrid:MXOnly-1U-NoLED
- MX84: value KC_ENT -> \; footprint MX_Alps_Hybrid:MXOnly-2.25U-NoLED -> MX_Alps_Hybrid:MXOnly-1.25U-NoLED
- MX85: value MO(1) -> Enter; footprint MX_Alps_Hybrid:MXOnly-1U-NoLED -> MX_Alps_Hybrid:MXOnly-2U-NoLED; moved to B.Cu
- MX86: value KC_DOWN -> Fn2
- MX87: value KC_DEL -> Up
- MX88: value KC_PGUP -> Down
- MX89: value KC_PGDN -> Page Up
- MX9: value KC_P2 -> PSLS
- MX90: value KC_UP -> Caps2; footprint MX_Alps_Hybrid:MXOnly-1U-NoLED -> MX_Alps_Hybrid:MXOnly-1.5U-NoLED
- MX91: value KC_RIGHT -> Page Down
- MX92: value KC_P0 -> Right; footprint MX_Alps_Hybrid:MXOnly-2U-ReversedStabilizers-NoLED -> MX_Alps_Hybrid:MXOnly-1U-NoLED
- moved D18 441.8 mm to (448.7, 288.7), turned to 0 degrees
- moved MX92 421.4 mm to (430.9, 76.2)
- moved D30 415.1 mm to (467.2, 275.5), turned to 0 degrees
- moved D35 400.9 mm to (467.2, 278.8), turned to 0 degrees
- moved D31 391.0 mm to (431.4, 288.7), turned to 0 degrees
- moved D36 387.3 mm to (467.2, 265.4), turned to 0 degrees
- moved D32 381.7 mm to (437.2, 292.0), turned to 0 degrees
- moved D39 367.9 mm to (426.0, 295.4), turned to 0 degrees
- moved D37 363.3 mm to (431.7, 295.4), turned to 0 degrees
- moved D44 353.3 mm to (420.2, 295.4), turned to 0 degrees
- moved D40 351.0 mm to (419.9, 288.7), turned to 0 degrees
- moved D38 335.7 mm to (425.7, 292.0), turned to 0 degrees
- moved D46 329.0 mm to (431.4, 292.0), turned to 0 degrees
- moved D45 328.2 mm to (408.4, 288.7), turned to 0 degrees
- moved D49 327.6 mm to (408.7, 295.4), turned to 0 degrees
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Connections:
- D10 pad 1: Row4 -> Row1
- D11 pad 1: Row0 -> Row2
- D12 pad 1: Row1 -> Row3
- D13 pad 1: Row2 -> Row4
- D14 pad 1: Row3 -> Row5
- D15 pad 1: Row4 -> Row6
- D16 pad 1: Row0 -> Row7
- D17 pad 1: Row2 -> Row0
- D18 pad 1: Row3 -> Row1
- D19 pad 1: Row4 -> Row2
- D20 pad 1: Row0 -> Row3
- D21 pad 1: Row1 -> Row4
- D22 pad 1: Row2 -> Row5
- D23 pad 1: Row3 -> Row6
- D24 pad 1: Row4 -> Row7
- D30 pad 1: Row0 -> Row5
- D31 pad 1: Row1 -> Row6
- D32 pad 1: Row2 -> Row7
- D33 pad 1: Row3 -> Row0
- D34 pad 1: Row4 -> Row1
- D35 pad 1: Row0 -> Row2
- D36 pad 1: Row1 -> Row3
- D37 pad 1: Row2 -> Row4
- D38 pad 1: Row3 -> Row5
- D39 pad 1: Row0 -> Row6
- D40 pad 1: Row1 -> Row7
- D41 pad 1: Row2 -> Row0
- D42 pad 1: Row3 -> Row1
- D43 pad 1: Row4 -> Row2
- D44 pad 1: Row0 -> Row3
- D45 pad 1: Row1 -> Row4
- D46 pad 1: Row2 -> Row5
- D47 pad 1: Row3 -> Row6
- D48 pad 1: Row4 -> Row7
- D53 pad 1: Row0 -> Row4
- D54 pad 1: Row1 -> Row5
- D55 pad 1: Row2 -> Row6
- D56 pad 1: Row3 -> Row7
- D57 pad 1: Row4 -> Row0
- D58 pad 1: Row0 -> Row1
- D59 pad 1: Row1 -> Row2
- D6 pad 1: Row0 -> Row5
- D60 pad 1: Row2 -> Row3
- D61 pad 1: Row3 -> Row4
- D62 pad 1: Row4 -> Row5
- D63 pad 1: Row0 -> Row6
- D64 pad 1: Row1 -> Row7
- D65 pad 1: Row2 -> Row0
- D66 pad 1: Row3 -> Row1
- D67 pad 1: Row4 -> Row2
- D68 pad 1: Row0 -> Row3
- D69 pad 1: Row1 -> Row4
- D7 pad 1: Row1 -> Row6
- D70 pad 1: Row3 -> Row5
- D71 pad 1: Row4 -> Row6
- D72 pad 1: Row0 -> Row7
- D73 pad 1: Row1 -> Row0
- D74 pad 1: Row2 -> Row1
- D75 pad 1: Row3 -> Row2
- D76 pad 1: Row4 -> Row3
- D77 pad 1: Row0 -> Row4
- D78 pad 1: Row1 -> Row5
- D79 pad 1: Row2 -> Row6
- D8 pad 1: Row2 -> Row7
- D80 pad 1: Row3 -> Row7
- D81 pad 1: Row4 -> Row0
- D82 pad 1: Row0 -> Row1
- D83 pad 1: Row1 -> Row2
- D84 pad 1: Row2 -> Row3
- D85 pad 1: Row3 -> Row4
- D86 pad 1: Row4 -> Row5
- D87 pad 1: Row0 -> Row6
- D88 pad 1: Row1 -> Row7
- D89 pad 1: Row2 -> Row1
- D9 pad 1: Row3 -> Row0
- D90 pad 1: Row3 -> Row0
- D91 pad 1: Row4 -> Row2
- MX11 pad 1: Col2 -> Col1
- MX12 pad 1: Col2 -> Col1
- MX13 pad 1: Col2 -> Col1
- MX14 pad 1: Col2 -> Col1
- MX15 pad 1: Col2 -> Col1
- MX16 pad 1: Col3 -> Col1
- MX17 pad 1: Col3 -> Col2
- MX18 pad 1: Col3 -> Col2
- MX19 pad 1: Col3 -> Col2
- MX20 pad 1: Col4 -> Col2
- MX21 pad 1: Col4 -> Col2
- MX22 pad 1: Col4 -> Col2
- MX23 pad 1: Col4 -> Col2
- MX24 pad 1: Col4 -> Col2
- MX25 pad 1: Col5 -> Col3
- MX26 pad 1: Col5 -> Col3
- MX27 pad 1: Col5 -> Col3
- MX28 pad 1: Col5 -> Col3
- MX29 pad 1: Col5 -> Col3
- MX30 pad 1: Col6 -> Col3
- MX31 pad 1: Col6 -> Col3
- MX32 pad 1: Col6 -> Col3
- MX33 pad 1: Col6 -> Col4
- MX34 pad 1: Col6 -> Col4
- MX35 pad 1: Col7 -> Col4
- MX36 pad 1: Col7 -> Col4
- MX37 pad 1: Col7 -> Col4
- MX38 pad 1: Col7 -> Col4
- MX39 pad 1: Col8 -> Col4
- MX40 pad 1: Col8 -> Col4
- MX41 pad 1: Col8 -> Col5
- MX42 pad 1: Col8 -> Col5
- MX43 pad 1: Col8 -> Col5
- MX44 pad 1: Col9 -> Col5
- MX45 pad 1: Col9 -> Col5
- MX46 pad 1: Col9 -> Col5
- MX47 pad 1: Col9 -> Col5
- MX48 pad 1: Col9 -> Col5
- MX49 pad 1: Col10 -> Col6
- MX50 pad 1: Col10 -> Col6
- MX51 pad 1: Col10 -> Col6
- MX52 pad 1: Col10 -> Col6
- MX53 pad 1: Col11 -> Col6
- MX54 pad 1: Col11 -> Col6
- MX55 pad 1: Col11 -> Col6
- MX56 pad 1: Col11 -> Col6
- MX57 pad 1: Col11 -> Col7
- MX58 pad 1: Col12 -> Col7
- MX59 pad 1: Col12 -> Col7
- MX6 pad 1: Col1 -> Col0
- MX60 pad 1: Col12 -> Col7
- MX61 pad 1: Col12 -> Col7
- MX62 pad 1: Col12 -> Col7
- MX63 pad 1: Col13 -> Col7
- MX64 pad 1: Col13 -> Col7
- MX65 pad 1: Col13 -> Col8
- MX66 pad 1: Col13 -> Col8
- MX67 pad 1: Col13 -> Col8
- MX68 pad 1: Col14 -> Col8
- MX69 pad 1: Col14 -> Col8
- MX7 pad 1: Col1 -> Col0
- MX70 pad 1: Col14 -> Col8
- MX71 pad 1: Col14 -> Col8
- MX72 pad 1: Col15 -> Col8
- MX73 pad 1: Col15 -> Col9
- MX74 pad 1: Col15 -> Col9
- MX75 pad 1: Col15 -> Col9
- MX76 pad 1: Col15 -> Col9
- MX77 pad 1: Col16 -> Col9
- MX78 pad 1: Col16 -> Col9
- MX79 pad 1: Col16 -> Col9
- MX8 pad 1: Col1 -> Col0
- MX80 pad 1: Col16 -> Col9
- MX81 pad 1: Col16 -> Col10
- MX82 pad 1: Col17 -> Col10
- MX83 pad 1: Col17 -> Col10
- MX84 pad 1: Col17 -> Col10
- MX85 pad 1: Col17 -> Col10
- MX86 pad 1: Col17 -> Col10
- MX87 pad 1: Col18 -> Col10
- MX88 pad 1: Col18 -> Col10
- MX89 pad 1: Col18 -> Col11
- MX90 pad 1: Col18 -> Col2
- MX90 pad 2: Net-(D90-Pad2) -> Net-(D22-Pad2)
- MX91 pad 1: Col18 -> Col11
- MX92 pad 1: Col0 -> Col11
- MX92 pad 2: Net-(D5-Pad2) -> Net-(D92-Pad2)
- U1 pad 10: Col7 -> Row6
- U1 pad 11: Col8 -> Net-(U1-Pad11)
- U1 pad 12: Col9 -> Net-(U1-Pad12)
- U1 pad 13: Col10 -> Row7
- U1 pad 14: Col11 -> Col6
- U1 pad 15: Col12 -> Col7
- U1 pad 16: Col13 -> Col8
- U1 pad 17: Col14 -> Col9
- U1 pad 18: Col15 -> Col10
- U1 pad 19: Col16 -> Col11
- U1 pad 20: Col17 -> EN2
- U1 pad 23: Net-(U1-Pad23) -> GND
- U1 pad 24: Col18 -> EN1
- U1 pad 9: Col6 -> Row5
Routing:
- net Row7: track 0.00 -> 337.2 mm, vias 0 -> 3
- net Col18: track 296.9 -> 0.00 mm
- net Row4: track 477.8 -> 183.5 mm, vias 1 -> 3
- net Row1: track 479.3 -> 195.9 mm
- net Col17: track 275.2 -> 0.00 mm
- net Col16: track 257.3 -> 0.00 mm
- net Row2: track 458.4 -> 222.7 mm, vias 1 -> 6
- net Row6: track 0.00 -> 228.0 mm, vias 0 -> 6
- net Col15: track 222.0 -> 0.00 mm
- net EN2: track 0.00 -> 215.3 mm
- net GND: track 0.00 -> 209.6 mm
- net Col14: track 208.0 -> 0.00 mm
- net EN1: track 0.00 -> 207.9 mm
- net Col10: track 84.0 -> 291.5 mm
- net Row3: track 465.2 -> 271.0 mm, vias 1 -> 2
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- removed copper zone on B.Cu, net (none)
- removed copper zone on F.Cu, net (none)
Other:
- board size 442.2 x 112.7 mm -> 458 x 99.2 mm

Commit message: Update PCB and gerber
Parts:
- MX85: moved to F.Cu
- moved D18 441.8 mm to (66.7, 66.6), turned to 270 degrees
- moved D35 418.5 mm to (133.1, 26.8), turned to 80 degrees
- moved D36 393.4 mm to (151.8, 30.2), turned to 80 degrees
- moved D32 383.6 mm to (141.5, 47.7), turned to 80 degrees
- moved D30 371.9 mm to (145.9, 88.2), turned to 80 degrees
- moved De 365.7 mm to (189.4, 36.8), turned to 80 degrees
- moved D37 365.2 mm to (160.2, 51.0), turned to 80 degrees
- moved D31 361.6 mm to (145.2, 67.7), turned to 80 degrees
- moved D43 355.2 mm to (170.6, 33.5), turned to 80 degrees
- moved D38 342.5 mm to (164.0, 71.0), turned to 80 degrees
- moved D44 341.0 mm to (179.0, 54.3), turned to 80 degrees
- moved D49 331.9 mm to (223.8, 19.7), turned to 100 degrees
- moved D46 331.0 mm to (197.8, 57.6), turned to 80 degrees
- moved D40 319.7 mm to (182.7, 74.3), turned to 80 degrees
- moved D39 311.1 mm to (188.3, 94.6), turned to 80 degrees
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- renumbered D47 to De
Routing:
- net Row3: track 271.0 -> 658.8 mm, vias 2 -> 14
- net Row1: track 195.9 -> 579.8 mm, vias 3 -> 8
- net Row6: track 228.0 -> 598.3 mm, vias 6 -> 12
- net Row4: track 183.5 -> 549.9 mm, vias 3 -> 14
- net Row5: track 176.2 -> 540.9 mm, vias 2 -> 11
- net Row2: track 222.7 -> 557.9 mm, vias 6 -> 3
- net Row7: track 337.2 -> 622.5 mm, vias 3 -> 16
- net Col5: track 1.78 -> 219.2 mm
- net Row0: track 254.7 -> 428.2 mm, vias 3 -> 0
- net Col7: track 33.6 -> 184.3 mm
- net Col6: track 29.6 -> 161.0 mm
- net Net-(D54-Pad2): track 0.00 -> 32.8 mm, vias 0 -> 1
- net Col8: track 259.7 -> 236.0 mm, vias 0 -> 1
- net Net-(D39-Pad2): track 0.00 -> 22.2 mm
- net Net-(D50-Pad2): track 0.00 -> 21.2 mm
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- added copper zone on B.Cu, net (none)
- added copper zone on F.Cu, net (none)
Other:
- board size 458 x 99.2 mm -> 450 x 112.6 mm

Commit message: Finished Edits
Parts:
- added H1: MountingHole, MountingHole:MountingHole_2.2mm_M2_Pad, F.Cu at (122.4, 38.2)
- added H11: MountingHole, MountingHole:MountingHole_2.2mm_M2_Pad, F.Cu at (395.6, 0.43)
- added H2: MountingHole, MountingHole:MountingHole_2.2mm_M2_Pad, F.Cu at (242.8, -4.51)
- added H3: MountingHole, MountingHole:MountingHole_2.2mm_M2_Pad, F.Cu at (303.6, 39.2)
- added H4: MountingHole, MountingHole:MountingHole_2.2mm_M2_Pad, F.Cu at (212.2, 48.5)
- added H5: MountingHole, MountingHole:MountingHole_2.2mm_M2_Pad, F.Cu at (212.2, 91.5)
- added H6: MountingHole, MountingHole:MountingHole_2.2mm_M2_Pad, F.Cu at (28.6, 0.43)
- added H7: MountingHole, MountingHole:MountingHole_2.2mm_M2_Pad, F.Cu at (38.8, 63.9)
- added H8: MountingHole, MountingHole:MountingHole_2.2mm_M2_Pad, F.Cu at (395.6, 63.9)
- added H9: MountingHole, MountingHole:MountingHole_2.2mm_M2_Pad, F.Cu at (179.6, -4.51)
- added TP1: TestPoint, TestPoint:TestPoint_Pad_1.0x1.0mm, B.Cu at (400.9, 45.0)
- added TP2: TestPoint, TestPoint:TestPoint_Pad_1.0x1.0mm, B.Cu at (400.9, 39.0)
- added TP3: TestPoint, TestPoint:TestPoint_Pad_1.0x1.0mm, B.Cu at (400.9, 42.0)
- MX90: footprint MX_Alps_Hybrid:MXOnly-1.5U-NoLED -> MX_Alps_Hybrid:MXOnly-1.25U-NoLED
- moved MX90 2.38 mm to (81.0, 38.1)
- renumbered De to D47
Connections:
- U1 pad 11: Net-(U1-Pad11) -> DataIn
- U1 pad 21: Net-(U1-Pad21) -> VCC
Routing:
- net DataIn: track 0.00 -> 288.4 mm, vias 0 -> 2
- net VCC: track 0.00 -> 243.9 mm, vias 0 -> 2
- net GND: track 209.6 -> 266.3 mm, vias 0 -> 2
- net Col2: track 299.4 -> 296.0 mm
- net Net-(D22-Pad2): track 16.8 -> 19.2 mm
- net Net-(U1-Pad21): track 1.78 -> 0.00 mm
- net Net-(U1-Pad11): track 1.78 -> 0.00 mm

Commit message: Final Update
Parts:
- removed TP1, TP2, TP3: TestPoint, TestPoint:TestPoint_Pad_1.0x1.0mm
- added OL1: OLED, kbd:OLED_v2, F.Cu at (408.0, 6.48)
- moved MX75 6.42 mm to (301.0, 18.2), turned to 10 degrees
- moved MX84 4.76 mm to (362.1, 19.1)
- moved MX76 4.76 mm to (321.6, 19.1)
- moved MX83 4.76 mm to (340.7, 19.1)
- moved H7 2.91 mm to (38.1, 66.7)
- moved MX73 2.38 mm to (309.7, -2.38)
Connections:
- U1 pad 11: DataIn -> Data1
- U1 pad 12: Net-(U1-Pad12) -> Data2
Routing:
- net DataIn: track 288.4 -> 0.00 mm, vias 2 -> 0
- net Data1: track 0.00 -> 230.1 mm
- net Data2: track 0.00 -> 228.4 mm
- net VCC: track 243.9 -> 197.6 mm, vias 2 -> 0
- net GND: track 266.3 -> 232.4 mm, vias 2 -> 0
- net Net-(D75-Pad2): track 21.4 -> 16.1 mm, vias 0 -> 1
- net Net-(D76-Pad2): track 21.4 -> 16.5 mm
- net Net-(D73-Pad2): track 19.0 -> 23.8 mm
- net Net-(D84-Pad2): track 18.8 -> 15.5 mm
- net Col9: track 265.5 -> 268.1 mm
- net Col10: track 297.4 -> 299.7 mm
- net Net-(U1-Pad12): track 2.01 -> 0.00 mm
- net Row0: track 428.2 -> 429.0 mm
- net Net-(D83-Pad2): track 21.4 -> 20.7 mm
- net Row7: track 622.5 -> 623.1 mm

Commit message: Fixing Errors
Routing:
- net Col2: track 296.0 -> 296.8 mm

Commit message: Update V2.kicad_pcb
Fixed Enter shift and space size
Parts:
- added MX78: RSHFT, MX_Alps_Hybrid:MXOnly-2.75U-NoLED, F.Cu at (354.9, 57.1)
- MX23, MX84: footprint MX_Alps_Hybrid:MXOnly-1.25U-NoLED -> MX_Alps_Hybrid:MXOnly-1.5U-NoLED
- MX85: footprint MX_Alps_Hybrid:MXOnly-2U-NoLED -> MX_Alps_Hybrid:MXOnly-2.25U-NoLED
- moved D18 39.2 mm to (66.7, 27.5)
- moved MX18 38.1 mm to (57.1, 28.6)
- moved MX19 38.1 mm to (57.1, 66.7)
- moved D19 20.3 mm to (66.7, 47.6), turned to 270 degrees
- moved D43 7.15 mm to (177.6, 34.7)
- moved MX43 7.14 mm to (169.5, 26.1)
- moved MX35 7.14 mm to (131.9, 19.4)
- moved MX36 7.14 mm to (150.7, 22.8)
- moved MX47 7.14 mm to (188.2, 29.4)
- moved D36 7.14 mm to (158.9, 31.4)
- moved D35 7.13 mm to (140.1, 28.1)
- moved D47 7.12 mm to (196.4, 38.0)
- moved MX26 4.76 mm to (107.2, 19.1)
- moved MX34 3.95 mm to (135.7, -2.38), turned to 0 degrees
- moved MX84 2.38 mm to (364.5, 19.1)
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Routing:
- net Row1: track 579.8 -> 519.9 mm, vias 8 -> 5
- net Row2: track 557.9 -> 571.4 mm, vias 3 -> 6
- net Col5: track 219.2 -> 207.5 mm
- net Col2: track 296.8 -> 305.1 mm
- net Col4: track 238.2 -> 231.8 mm
- net Net-(D19-Pad2): track 14.8 -> 20.9 mm
- net Net-(D34-Pad2): track 13.7 -> 18.8 mm
- net Col9: track 268.1 -> 272.9 mm
- net Net-(D78-Pad2): track 29.3 -> 34.1 mm
- net Row5: track 540.9 -> 536.6 mm
- net Row6: track 598.3 -> 602.5 mm
- net Net-(D24-Pad2): track 15.8 -> 18.2 mm
- net Net-(D85-Pad2): track 27.0 -> 29.3 mm
- net Net-(D26-Pad2): track 15.8 -> 13.9 mm
- net Net-(D33-Pad2): track 15.8 -> 13.9 mm
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