File: V2/V2.sch (KiCad schematic (older format))
At the start: 199 parts, among them SW1 Rotary_Encoder_Switch, U1 Elite-C

Commit message: Final Update
Parts:
- removed TP1, TP2, TP3: TestPoint, TestPoint:TestPoint_Pad_1.0x1.0mm, symbol Connector:TestPoint
- added OL1: OLED, kbd:OLED_v2, symbol kbd:OLED
Connections:
- net GND: now also OL1.4 (GND)
- net VCC: now also OL1.3 (VCC)
- net Data2: now reaches U1.12 (9/PB5)
- net Data2: now also OL1.2 (SCL)
- net DataIn renamed Data1
- net Data1: now also OL1.1 (SDA)
Changed lines of the file:
@@
 $EndComp
 $Comp
-L Connector:TestPoint TP1
-U 1 1 6133C5CF
-P 3450 6625
-F 0 "TP1" H 3508 6743 50  0000 L CNN
-F 1 "TestPoint" H 3508 6652 50  0000 L CNN
-F 2 "TestPoint:TestPoint_Pad_1.0x1.0mm" H 3650 6625 50  0001 C CNN
-F 3 "~" H 3650 6625 50  0001 C CNN
-	1    3450 6625
-	1    0    0    -1
-$EndComp
-$Comp
-L Connector:TestPoint TP2
-U 1 1 6133CCCC
-P 3450 6975
-F 0 "TP2" H 3508 7093 50  0000 L CNN
-F 1 "TestPoint" H 3508 7002 50  0000 L CNN
-F 2 "TestPoint:TestPoint_Pad_1.0x1.0mm" H 3650 6975 50  0001 C CNN
-F 3 "~" H 3650 6975 50  0001 C CNN
-	1    3450 6975
-	1    0    0    -1
-$EndComp
-$Comp
-L Connector:TestPoint TP3
-U 1 1 6133CF80
-P 3450 7425
-F 0 "TP3" H 3508 7543 50  0000 L CNN
-F 1 "TestPoint" H 3508 7452 50  0000 L CNN
-F 2 "TestPoint:TestPoint_Pad_1.0x1.0mm" H 3650 7425 50  0001 C CNN
-F 3 "~" H 3650 7425 50  0001 C CNN
-	1    3450 7425
-	1    0    0    -1
-$EndComp
-$Comp
-L helix-cache:GND #PWR?
+L helix-cache:GND #PWR03
 U 1 1 6134E6F1
-P 3450 6625
-F 0 "#PWR?" H 3450 6375 50  0001 C CNN
-F 1 "GND" V 3455 6497 50  0000 R CNN
-F 2 "" H 3450 6625 50  0000 C CNN
-F 3 "" H 3450 6625 50  0000 C CNN
-	1    3450 6625
+P 1425 6825
+F 0 "#PWR03" H 1425 6575 50  0001 C CNN
+F 1 "GND" V 1430 6697 50  0000 R CNN
+F 2 "" H 1425 6825 50  0000 C CNN
+F 3 "" H 1425 6825 50  0000 C CNN
+	1    1425 6825
 	1    0    0    -1
 $EndComp
 Text GLabel 2150 1125 2    50   Input ~ 0
 VCC
-Text GLabel 3450 6975 0    50   Input ~ 0
+Text GLabel 1425 6675 0    50   Input ~ 0
 VCC
 Text GLabel 750  1825 0    50   Input ~ 0
-DataIn
-Text GLabel 3450 7425 0    50   Input ~ 0
-DataIn
+Data1
+Text GLabel 1425 6375 0    50   Input ~ 0
+Data1
+$Comp
+L kbd:OLED OL1
+U 1 1 613000F0
+P 2175 6625
+F 0 "OL1" H 2803 6694 51  0000 L CNN
+F 1 "OLED" H 2803 6604 47  0000 L CNN
+F 2 "kbd:OLED_v2" H 2175 6725 60  0001 C CNN
+F 3 "" H 2175 6725 60  0001 C CNN
+	1    2175 6625
+	1    0    0    -1
+$EndComp
+Text GLabel 1425 6525 0    50   Input ~ 0
+Data2
+Text GLabel 750  1925 0    50   Input ~ 0
+Data2
 $EndSCHEMATC
